File: O'Shambles/pcb/KiCad Files/O'Shambles.kicad_pcb (KiCad board)
At the start: 2 copper layers, 258.1 x 119.5 mm, 130 parts, among them SW1 Rotary_Encoder_Switch, SW10 SW_PUSH, SW11 SW_PUSH, SW12 SW_PUSH, SW13 SW_PUSH, SW14 SW_PUSH, SW15 SW_PUSH, SW16 SW_PUSH, SW17 SW_PUSH, SW18 SW_PUSH, SW19 SW_PUSH, SW2 Rotary_Encoder_Switch, SW20 SW_PUSH, SW21 SW_PUSH, SW22 SW_PUSH, SW23 SW_PUSH, SW24 SW_PUSH, SW25 SW_PUSH, SW26 SW_PUSH, SW27 SW_PUSH, SW28 SW_PUSH, SW29 SW_PUSH, SW3 SW_PUSH, SW30 SW_PUSH, SW31 SW_PUSH, SW32 SW_PUSH, SW33 SW_PUSH, SW34 SW_PUSH, SW35 SW_PUSH, SW36 SW_PUSH, SW37 SW_PUSH, SW38 SW_PUSH, SW39 SW_PUSH, SW4 SW_PUSH, SW40 SW_PUSH, SW41 SW_PUSH, SW42 SW_PUSH, SW43 SW_PUSH, SW44 SW_PUSH, SW45 SW_PUSH, SW46 SW_PUSH, SW47 SW_PUSH, SW48 SW_PUSH, SW49 SW_PUSH, SW5 SW_PUSH, SW50 SW_PUSH, SW51 SW_PUSH, SW52 SW_PUSH, SW53 SW_PUSH, SW54 SW_PUSH, SW55 SW_PUSH, SW56 SW_PUSH, SW57 SW_PUSH, SW58 SW_PUSH, SW59 SW_PUSH, SW6 SW_PUSH, SW60 SW_PUSH, SW61 SW_PUSH, SW62 SW_PUSH, SW63 SW_PUSH, SW64 SW_PUSH, SW65 SW_PUSH, SW7 SW_PUSH, SW8 SW_PUSH, SW9 SW_PUSH, U1 ProMicro, U2 ProMicro

Commit message: blockhead two, no ave, and some other boards
Parts:
- added H1: MountingHole, keyboard_parts:HOLE_M3, F.Cu at (39.1, 135.5)
- added H2: MountingHole, keyboard_parts:HOLE_M3, F.Cu at (48.6, 76.0)
- added H3: MountingHole, keyboard_parts:HOLE_M3, F.Cu at (115.3, 76.0)
- added H4: MountingHole, keyboard_parts:HOLE_M3, F.Cu at (248.6, 76.0)
- added H5: MountingHole, keyboard_parts:HOLE_M3, F.Cu at (110.5, 137.9)
- added H6: MountingHole, keyboard_parts:HOLE_M3, F.Cu at (253.4, 137.9)
- added H7: MountingHole, keyboard_parts:HOLE_M3, F.Cu at (181.9, 116.5)
- moved D61 3.86 mm to (44.9, 135.6)
- moved SW2 1.21 mm to (48.9, 95.0)
Routing:
- net ROW2: track 434.4 -> 438.0 mm
- net COL8: track 778.8 -> 782.1 mm
- net Net-(D61-Pad2): track 27.7 -> 24.6 mm
- net COL6: track 744.7 -> 747.7 mm
- net COL5: track 680.3 -> 683.2 mm
- net Row2Diode: track 37.6 -> 35.4 mm
- net ROW1: track 483.1 -> 484.9 mm
- net COL7: track 481.9 -> 483.4 mm
- net COL3: track 600.5 -> 601.9 mm
- net COL4: track 635.1 -> 633.9 mm
- net COL2: track 524.7 -> 525.9 mm
- net R1: track 307.2 -> 308.3 mm
- net R2: track 297.7 -> 298.5 mm
- net GND: track 369.3 -> 370.1 mm
- net COL1: track 509.6 -> 510.1 mm
